File: PCB/Watch1.1/Watch1.1.sch (EAGLE design)
At the start: 27 parts, among them CN4 FTDI, IC1 LM358D, U1 ATMega-328, Y1 32.768kHz

Commit message: fix diode position
Connections:
- net A6: now also D1.C
- net N$14: no longer D1.C
Changed lines of the file:
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@@
 <setting verticaltext="up"/>
 </settings>
-<grid distance="0.1" unitdist="inch" unit="inch" style="lines" multiple="1" display="no" altdistance="0.01" altunitdist="inch" altunit="inch"/>
+<grid distance="0.05" unitdist="inch" unit="inch" style="lines" multiple="1" display="no" altdistance="0.01" altunitdist="inch" altunit="inch"/>
 <layers>
 <layer number="1" name="Top" color="4" fill="1" visible="no" active="no"/>
@@
 <junction x="161.29" y="57.15"/>
 <label x="165.1" y="57.15" size="1.778" layer="95"/>
+<pinref part="D1" gate="G$1" pin="C"/>
+<wire x1="153.67" y1="50.8" x2="153.67" y2="57.15" width="0.1524" layer="91"/>
+<wire x1="153.67" y1="57.15" x2="161.29" y2="57.15" width="0.1524" layer="91"/>
 </segment>
 </net>
@@
 </segment>
 </net>
+<net name="N$13" class="0">
+<segment>
+<pinref part="U1" gate="G$1" pin="PB7(XTAL2/TOSC2)"/>
+<wire x1="31.75" y1="119.38" x2="30.48" y2="119.38" width="0.1524" layer="91"/>
+<pinref part="Y1" gate="G$1" pin="1"/>
+<wire x1="30.48" y1="109.22" x2="30.48" y2="119.38" width="0.1524" layer="91"/>
+</segment>
+</net>
 <net name="N$14" class="0">
 <segment>
@@
 <wire x1="161.29" y1="71.12" x2="161.29" y2="74.93" width="0.1524" layer="91"/>
 <pinref part="SV1" gate="G$1" pin="2"/>
-<wire x1="161.29" y1="74.93" x2="153.67" y2="74.93" width="0.1524" layer="91"/>
-<pinref part="D1" gate="G$1" pin="C"/>
-<wire x1="153.67" y1="74.93" x2="144.78" y2="74.93" width="0.1524" layer="91"/>
+<wire x1="161.29" y1="74.93" x2="144.78" y2="74.93" width="0.1524" layer="91"/>
 <wire x1="144.78" y1="74.93" x2="129.54" y2="74.93" width="0.1524" layer="91"/>
-<wire x1="153.67" y1="50.8" x2="153.67" y2="74.93" width="0.1524" layer="91"/>
-<junction x="153.67" y="74.93"/>
 <pinref part="C3" gate="G$1" pin="1"/>
 <wire x1="144.78" y1="63.5" x2="144.78" y2="66.04" width="0.1524" layer="91"/>
@@
 </segment>
 </net>
-<net name="N$13" class="0">
-<segment>
-<pinref part="U1" gate="G$1" pin="PB7(XTAL2/TOSC2)"/>
-<wire x1="31.75" y1="119.38" x2="30.48" y2="119.38" width="0.1524" layer="91"/>
-<pinref part="Y1" gate="G$1" pin="1"/>
-<wire x1="30.48" y1="109.22" x2="30.48" y2="119.38" width="0.1524" layer="91"/>
-</segment>
-</net>

Commit message: adjustments
Parts:
- removed R12: 1k5, LowPowerLab:RESISTOR0805
- removed R13: 2k, LowPowerLab:RESISTOR0805
- removed R14: 10k, LowPowerLab:RESISTOR0805
- added R6: 1r, LowPowerLab:RESISTOR0805
- added R7: 1k5, LowPowerLab:RESISTOR0805
- added R8: 12k, LowPowerLab:RESISTOR0805
- R10: value 1k5 -> 2k
- R11: value 12k -> 10k
- R2, R3, R4, R5: value 82r -> 330r
- R9: value 1r -> 1k5
- renumbered SV1 to CN1, U$1 to CN2
Connections:
- net A6: now also R10.2, R11.1; no longer R13.2, R14.1
- net A7: now also R9.1; no longer R12.1
- net GND: now also R6.1, R7.1; no longer R13.1, R9.1
- net N$11: now also R8.1, R9.2; no longer R11.1, R12.2
- net N$14: now also R11.2; no longer R14.2
- net N$8: now also R6.2; no longer R9.2
- net N$9: now also R7.2, R8.2; no longer R10.2, R11.2
Other:
- moved on the sheet: R10, R11, R9
Changed lines of the file:
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@@
 <setting verticaltext="up"/>
 </settings>
-<grid distance="0.05" unitdist="inch" unit="inch" style="lines" multiple="1" display="no" altdistance="0.01" altunitdist="inch" altunit="inch"/>
+<grid distance="0.1" unitdist="inch" unit="inch" style="lines" multiple="1" display="no" altdistance="0.01" altunitdist="inch" altunit="inch"/>
 <layers>
 <layer number="1" name="Top" color="4" fill="1" visible="no" active="no"/>
@@
 <class number="0" name="default" width="0" drill="0">
 </class>
-<class number="1" name="power" width="0.381" drill="0">
+<class number="1" name="power" width="0.508" drill="0">
 <clearance class="1" value="0.254"/>
 </class>
@@
 <part name="CN4" library="pinhead" deviceset="PINHD-1X6" device="" value="FTDI"/>
 <part name="LED1" library="playground" deviceset="HP_DISPLAY" device=""/>
-<part name="R2" library="LowPowerLab" deviceset="RESISTOR" device="0805" value="82r"/>
-<part name="R3" library="LowPowerLab" deviceset="RESISTOR" device="0805" value="82r"/>
-<part name="R4" library="LowPowerLab" deviceset="RESISTOR" device="0805" value="82r"/>
-<part name="R5" library="LowPowerLab" deviceset="RESISTOR" device="0805" value="82r"/>
+<part name="R2" library="LowPowerLab" deviceset="RESISTOR" device="0805" value="330r"/>
+<part name="R3" library="LowPowerLab" deviceset="RESISTOR" device="0805" value="330r"/>
+<part name="R4" library="LowPowerLab" deviceset="RESISTOR" device="0805" value="330r"/>
+<part name="R5" library="LowPowerLab" deviceset="RESISTOR" device="0805" value="330r"/>
 <part name="IC1" library="linear" deviceset="LM358" device="D"/>
-<part name="R9" library="LowPowerLab" deviceset="RESISTOR" device="0805" value="1r"/>
-<part name="R10" library="LowPowerLab" deviceset="RESISTOR" device="0805" value="1k5"/>
-<part name="R11" library="LowPowerLab" deviceset="RESISTOR" device="0805" value="12k"/>
-<part name="R12" library="LowPowerLab" deviceset="RESISTOR" device="0805" value="1k5"/>
+<part name="R6" library="LowPowerLab" deviceset="RESISTOR" device="0805" value="1r"/>
+<part name="R7" library="LowPowerLab" deviceset="RESISTOR" device="0805" value="1k5"/>
+<part name="R8" library="LowPowerLab" deviceset="RESISTOR" device="0805" value="12k"/>
+<part name="R9" library="LowPowerLab" deviceset="RESISTOR" device="0805" value="1k5"/>
 <part name="SUPPLY8" library="supply2" deviceset="GND" device=""/>
-<part name="SV1" library="con-lstb" deviceset="MA03-1" device=""/>
+<part name="CN1" library="con-lstb" deviceset="MA03-1" device=""/>
 <part name="SUPPLY10" library="supply2" deviceset="GND" device=""/>
 <part name="SUPPLY11" library="supply2" deviceset="GND" device=""/>
-<part name="R13" library="LowPowerLab" deviceset="RESISTOR" device="0805" value="2k"/>
-<part name="R14" library="LowPowerLab" deviceset="RESISTOR" device="0805" value="10k"/>
+<part name="R10" library="LowPowerLab" deviceset="RESISTOR" device="0805" value="2k"/>
+<part name="R11" library="LowPowerLab" deviceset="RESISTOR" device="0805" value="10k"/>
 <part name="D1" library="diode" deviceset="BZX84CSMD" device=""/>
 <part name="PTC" library="rcl" deviceset="R-US_" device="R1206" value="500ma"/>
@@
 <part name="SUPPLY15" library="SparkFun" deviceset="VCC" device="" value="3.3V"/>
 <part name="BAT1" library="SparkFun-Electromechanical" deviceset="BATTERY" device="20MM_4LEGS_OVERPASTE" value="20mm coincell"/>
-<part name="U$1" library="Richard1" deviceset="3PIN-HEADER-RA" device=""/>
+<part name="CN2" library="Richard1" deviceset="3PIN-HEADER-RA" device=""/>
 <part name="SUPPLY2" library="SparkFun" deviceset="VCC" device="" value="3.3V"/>
 <part name="SUPPLY16" library="supply2" deviceset="GND" device=""/>
@@
 <instance part="R5" gate="G$1" x="241.3" y="113.03" rot="R90"/>
 <instance part="IC1" gate="A" x="203.2" y="74.93"/>
-<instance part="R9" gate="G$1" x="180.34" y="55.88" rot="R90"/>
-<instance part="R10" gate="G$1" x="193.04" y="55.88" rot="R90"/>
-<instance part="R11" gate="G$1" x="209.55" y="62.23" rot="R180"/>
-<instance part="R12" gate="G$1" x="224.79" y="62.23" rot="R180"/>
+<instance part="R6" gate="G$1" x="180.34" y="55.88" rot="R90"/>
+<instance part="R7" gate="G$1" x="193.04" y="55.88" rot="R90"/>
+<instance part="R8" gate="G$1" x="209.55" y="62.23" rot="R180"/>
+<instance part="R9" gate="G$1" x="224.79" y="62.23" rot="R180"/>
 <instance part="SUPPLY8" gate="GND" x="180.34" y="40.64"/>
-<instance part="SV1" gate="G$1" x="121.92" y="74.93"/>
+<instance part="CN1" gate="G$1" x="121.92" y="74.93"/>
 <instance part="SUPPLY10" gate="GND" x="135.89" y="53.34"/>
 <instance part="SUPPLY11" gate="GND" x="161.29" y="35.56"/>
-<instance part="R13" gate="G$1" x="161.29" y="48.26" rot="R90"/>
-<instance part="R14" gate="G$1" x="161.29" y="66.04" rot="R90"/>
+<instance part="R10" gate="G$1" x="161.29" y="48.26" rot="R90"/>
+<instance part="R11" gate="G$1" x="161.29" y="66.04" rot="R90"/>
 <instance part="D1" gate="G$1" x="153.67" y="48.26" rot="R90"/>
 <instance part="PTC" gate="G$1" x="168.91" y="77.47"/>
@@
 <instance part="SUPPLY15" gate="1" x="237.49" y="54.61"/>
 <instance part="BAT1" gate="G$1" x="237.49" y="43.18" rot="R270"/>
-<instance part="U$1" gate="G$1" x="144.78" y="92.71" rot="R90"/>
+<instance part="CN2" gate="G$1" x="144.78" y="92.71" rot="R90"/>
 <instance part="IC1" gate="B" x="203.2" y="90.17"/>
 <instance part="IC1" gate="P" x="247.65" y="78.74"/>
@@
 </segment>
 <segment>
-<pinref part="R9" gate="G$1" pin="1"/>
+<pinref part="R6" gate="G$1" pin="1"/>
 <pinref part="SUPPLY8" gate="GND" pin="GND"/>
 <wire x1="180.34" y1="50.8" x2="180.34" y2="46.99" width="0.1524" layer="91"/>
-<pinref part="R10" gate="G$1" pin="1"/>
+<pinref part="R7" gate="G$1" pin="1"/>
 <wire x1="180.34" y1="46.99" x2="180.34" y2="43.18" width="0.1524" layer="91"/>
 <wire x1="193.04" y1="50.8" x2="193.04" y2="46.99" width="0.1524" layer="91"/>
@@
 </segment>
 <segment>
-<pinref part="SV1" gate="G$1" pin="1"/>
+<pinref part="CN1" gate="G$1" pin="1"/>
 <pinref part="SUPPLY10" gate="GND" pin="GND"/>
 <wire x1="129.54" y1="72.39" x2="135.89" y2="72.39" width="0.1524" layer="91"/>
 <wire x1="135.89" y1="72.39" x2="135.89" y2="55.88" width="0.1524" layer="91"/>
-<pinref part="U$1" gate="G$1" pin="1"/>
+<pinref part="CN2" gate="G$1" pin="1"/>
 <wire x1="142.24" y1="82.55" x2="142.24" y2="72.39" width="0.1524" layer="91"/>
 <wire x1="142.24" y1="72.39" x2="135.89" y2="72.39" width="0.1524" layer="91"/>
@@
 </segment>
 <segment>
-<pinref part="R13" gate="G$1" pin="1"/>
+<pinref part="R10" gate="G$1" pin="1"/>
 <pinref part="SUPPLY11" gate="GND" pin="GND"/>
 <wire x1="161.29" y1="43.18" x2="161.29" y2="40.64" width="0.1524" layer="91"/>
@@
 </segment>
 <segment>
-<pinref part="R12" gate="G$1" pin="1"/>
+<pinref part="R9" gate="G$1" pin="1"/>
 <wire x1="229.87" y1="62.23" x2="233.68" y2="62.23" width="0.1524" layer="91"/>
 <wire x1="233.68" y1="62.23" x2="233.68" y2="74.93" width="0.1524" layer="91"/>
@@
 </segment>
 <segment>
-<pinref part="R13" gate="G$1" pin="2"/>
-<pinref part="R14" gate="G$1" pin="1"/>
+<pinref part="R10" gate="G$1" pin="2"/>
+<pinref part="R11" gate="G$1" pin="1"/>
 <wire x1="161.29" y1="53.34" x2="161.29" y2="57.15" width="0.1524" layer="91"/>
 <wire x1="161.29" y1="57.15" x2="161.29" y2="60.96" width="0.1524" layer="91"/>
@@
 </segment>
 </net>
-<net name="N$8" class="0">
-<segment>
-<pinref part="R9" gate="G$1" pin="2"/>
+<net name="N$8" class="1">
+<segment>
+<pinref part="R6" gate="G$1" pin="2"/>
 <wire x1="180.34" y1="60.96" x2="180.34" y2="77.47" width="0.1524" layer="91"/>
 <pinref part="IC1" gate="A" pin="+IN"/>
@@
 <segment>
 <pinref part="IC1" gate="A" pin="-IN"/>
-<pinref part="R10" gate="G$1" pin="2"/>
+<pinref part="R7" gate="G$1" pin="2"/>
 <wire x1="195.58" y1="72.39" x2="193.04" y2="72.39" width="0.1524" layer="91"/>
 <wire x1="193.04" y1="72.39" x2="193.04" y2="62.23" width="0.1524" layer="91"/>
-<pinref part="R11" gate="G$1" pin="2"/>
+<pinref part="R8" gate="G$1" pin="2"/>
 <wire x1="193.04" y1="62.23" x2="193.04" y2="60.96" width="0.1524" layer="91"/>
 <wire x1="204.47" y1="62.23" x2="193.04" y2="62.23" width="0.1524" layer="91"/>
@@
 <net name="N$11" class="0">
 <segment>
-<pinref part="R12" gate="G$1" pin="2"/>
-<pinref part="R11" gate="G$1" pin="1"/>
+<pinref part="R9" gate="G$1" pin="2"/>
+<pinref part="R8" gate="G$1" pin="1"/>
 <wire x1="219.71" y1="62.23" x2="214.63" y2="62.23" width="0.1524" layer="91"/>
 </segment>
 </net>
-<net name="N$7" class="0">
+<net name="N$7" class="1">
 <segment>
 <wire x1="163.83" y1="77.47" x2="137.16" y2="77.47" width="0.1524" layer="91"/>
-<pinref part="SV1" gate="G$1" pin="3"/>
+<pinref part="CN1" gate="G$1" pin="3"/>
 <pinref part="PTC" gate="G$1" pin="1"/>
-<pinref part="U$1" gate="G$1" pin="3"/>
+<pinref part="CN2" gate="G$1" pin="3"/>
 <wire x1="137.16" y1="77.47" x2="129.54" y2="77.47" width="0.1524" layer="91"/>
 <wire x1="137.16" y1="82.55" x2="137.16" y2="77.47" width="0.1524" layer="91"/>
@@
 <net name="N$14" class="0">
 <segment>
-<pinref part="R14" gate="G$1" pin="2"/>
+<pinref part="R11" gate="G$1" pin="2"/>
 <wire x1="161.29" y1="71.12" x2="161.29" y2="74.93" width="0.1524" layer="91"/>
-<pinref part="SV1" gate="G$1" pin="2"/>
+<pinref part="CN1" gate="G$1" pin="2"/>
 <wire x1="161.29" y1="74.93" x2="144.78" y2="74.93" width="0.1524" layer="91"/>
 <wire x1="144.78" y1="74.93" x2="129.54" y2="74.93" width="0.1524" layer="91"/>
@@
 <wire x1="139.7" y1="66.04" x2="144.78" y2="66.04" width="0.1524" layer="91"/>
 <junction x="144.78" y="66.04"/>
-<pinref part="U$1" gate="G$1" pin="2"/>
-</segment>
-</net>
+<pinref part="CN2" gate="G$1" pin="2"/>
+</segment>
+</net>
